File: pcb/balancebot.kicad_pcb (KiCad board)
At the start: 2 copper layers, 51.8 x 58.5 mm, 33 parts, among them J1 Conn_01x04, J2 Conn_01x02, J3 Conn_01x03, J4 Conn_01x04, J5 Conn_01x04, J6 Conn_01x07, U1 LSM6DS3, U2 DRV8835, U3 ESP32mini, U4 DSN-MINI-360

Commit message: Start using LSM6DS3 driver from mjstn/MarkWorldCodeModules.
Other:
- rule pad_to_mask_clearance: 0.2 -> -0.2
Changed lines of the file:
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@@
     (pad_size 0.9 0.9)
     (pad_drill 0.3)
-    (pad_to_mask_clearance 0.2)
+    (pad_to_mask_clearance -0.2)
     (aux_axis_origin 0 0)
     (visible_elements FFFFFF7F)
     (pcbplotparams
-      (layerselection 0x010fc_ffffffff)
+      (layerselection 0x01008_7ffffffe)
       (usegerberextensions false)
       (usegerberattributes false)
@@
       (padsonsilk false)
       (subtractmaskfromsilk false)
-      (outputformat 1)
+      (outputformat 5)
       (mirror false)
       (drillshape 0)
